File: hardware/esp32-wrover-breakout.sch (KiCad schematic (older format))
At the start: 1 part

Commit message: Schematic ready
Parts:
- added C? (x2): 0.1uF, symbol Device:C_Small
- added C? (x2): 10uF, symbol Device:C_Small
- added J?: Conn_01x05_Male, symbol Connector:Conn_01x05_Male
- added J? (x2): Conn_01x10_Male, symbol Connector:Conn_01x10_Male
- added Q? (x2): MUN5214DW1T1G, On_Semiconductor-MUN5214DW1T1G-*, symbol MUN5214DW1T1G:MUN5214DW1T1G
- added U?: XC6220B331MR, Package_TO_SOT_SMD:SOT-23-5, symbol Regulator_Linear:XC6220B331MR
Connections:
- net labels added: +3.3V, +5V, DTR, GND, GPIO0, GPIO14, GPIO15, GPIO18, GPIO19, GPIO21, GPIO22, GPIO23, GPIO25, GPIO26, GPIO27, GPIO32, GPIO33, GPIO35, GPIO4, GPIO5, RESET, RTS, RX, TX
- wire segments 0 -> 102
Other:
- moved on the sheet: IC?

Commit message: PCB placement and silkscreen done
Parts:
- C1, C4: renamed from C?; footprint (none) -> Capacitor_SMD:C_0805_2012Metric_Pad1.18x1.45mm_HandSolder
- C2, C3: renamed from C?; footprint (none) -> Capacitor_SMD:C_0603_1608Metric_Pad1.08x0.95mm_HandSolder
- J1: renamed from J?; value Conn_01x05_Male -> Conn_01x04_Male; footprint (none) -> Connector_PinHeader_2.54mm:PinHeader_1x04_P2.54mm_Vertical; symbol Connector:Conn_01x05_Male -> Connector:Conn_01x04_Male
- J2, J3: renamed from J?; footprint (none) -> Connector_PinHeader_2.54mm:PinHeader_1x10_P2.54mm_Vertical
- Q1: renamed from Q?; footprint On_Semiconductor-MUN5214DW1T1G-* -> MUN5214DW1T1G:On_Semiconductor-MUN5214DW1T1G-Manufacturer_Recommended
- gave numbers to parts that had none: 2
Connections:
- wire segments 102 -> 103
Changed lines of the file:
@@
 $EndDescr
 $Comp
-L ESP32-WROVER-E_M213EH6464PH3Q0:ESP32-WROVER-E_M213EH6464PH3Q0_ IC?
+L ESP32-WROVER-E_M213EH6464PH3Q0:ESP32-WROVER-E_M213EH6464PH3Q0_ IC1
 U 1 1 5FE6A6FF
 P 2750 3800
-F 0 "IC?" H 3500 4065 50  0000 C CNN
+F 0 "IC1" H 3500 4065 50  0000 C CNN
 F 1 "ESP32-WROVER-E_M213EH6464PH3Q0_" H 3500 3974 50  0000 C CNN
 F 2 "ESP32WROVEREM213EH6464PH3Q0" H 4100 3900 50  0001 L CNN
@@
 $EndComp
 $Comp
-L MUN5214DW1T1G:MUN5214DW1T1G Q?
+L MUN5214DW1T1G:MUN5214DW1T1G Q1
 U 2 1 5FE8E343
 P 8000 2550
-F 0 "Q?" H 8544 2596 50  0000 L CNN
+F 0 "Q1" H 8544 2596 50  0000 L CNN
 F 1 "MUN5214DW1T1G" H 8544 2505 50  0000 L CNN
-F 2 "On_Semiconductor-MUN5214DW1T1G-*" H 8000 3150 50  0001 L CNN
+F 2 "MUN5214DW1T1G:On_Semiconductor-MUN5214DW1T1G-Manufacturer_Recommended" H 8000 3150 50  0001 L CNN
 F 3 "http://www.onsemi.cn/pub_link/Collateral/DTC114YD-D.PDF" H 8000 3250 50  0001 L CNN
 F 4 "Manufacturer URL" H 8000 3350 50  0001 L CNN "Component Link 1 Description"
@@
 	1    0    0    1
 $EndComp
-Text Label 7450 3950 0    50   ~ 0
+Text Label 7450 4050 0    50   ~ 0
 RX
 Wire Wire Line
-	7650 3950 7450 3950
-Wire Wire Line
 	7650 4050 7450 4050
 Wire Wire Line
@@
 Wire Wire Line
 	7650 4350 7450 4350
-Text Label 7450 4350 0    50   ~ 0
-GND
 $Comp
 L power:GND #PWR0101
@@
 	4350 6150 4350 6000
 Connection ~ 4350 6000
-Text Label 7450 4050 0    50   ~ 0
+Text Label 7450 4150 0    50   ~ 0
 TX
-Text Label 7450 4150 0    50   ~ 0
+Text Label 7450 4250 0    50   ~ 0
 RTS
-Text Label 7450 4250 0    50   ~ 0
+Text Label 7450 4350 0    50   ~ 0
 DTR
 Text Label 4350 4700 0    50   ~ 0
@@
 TX
 $Comp
-L Device:C_Small C?
+L Device:C_Small C3
 U 1 1 5FF3A196
 P 2300 4150
-F 0 "C?" H 2392 4196 50  0000 L CNN
+F 0 "C3" H 2392 4196 50  0000 L CNN
 F 1 "0.1uF" H 2392 4105 50  0000 L CNN
-F 2 "" H 2300 4150 50  0001 C CNN
+F 2 "Capacitor_SMD:C_0603_1608Metric_Pad1.08x0.95mm_HandSolder" H 2300 4150 50  0001 C CNN
 F 3 "~" H 2300 4150 50  0001 C CNN
 	1    2300 4150
@@
 RESET
 $Comp
-L MUN5214DW1T1G:MUN5214DW1T1G Q?
+L MUN5214DW1T1G:MUN5214DW1T1G Q1
 U 1 1 5FE8C204
 P 8000 1700
-F 0 "Q?" H 8544 1746 50  0000 L CNN
+F 0 "Q1" H 8544 1746 50  0000 L CNN
 F 1 "MUN5214DW1T1G" H 8544 1655 50  0000 L CNN
-F 2 "On_Semiconductor-MUN5214DW1T1G-*" H 8000 2300 50  0001 L CNN
+F 2 "MUN5214DW1T1G:On_Semiconductor-MUN5214DW1T1G-Manufacturer_Recommended" H 8000 2300 50  0001 L CNN
 F 3 "http://www.onsemi.cn/pub_link/Collateral/DTC114YD-D.PDF" H 8000 2400 50  0001 L CNN
 F 4 "Manufacturer URL" H 8000 2500 50  0001 L CNN "Component Link 1 Description"
@@
 DTR
 $Comp
-L Device:C_Small C?
+L Device:C_Small C1
 U 1 1 5FFB1EE5
 P 1250 1600
-F 0 "C?" H 1342 1646 50  0000 L CNN
+F 0 "C1" H 1342 1646 50  0000 L CNN
 F 1 "10uF" H 1342 1555 50  0000 L CNN
-F 2 "" H 1250 1600 50  0001 C CNN
+F 2 "Capacitor_SMD:C_0805_2012Metric_Pad1.18x1.45mm_HandSolder" H 1250 1600 50  0001 C CNN
 F 3 "~" H 1250 1600 50  0001 C CNN
 	1    1250 1600
@@
 $EndComp
 $Comp
-L Device:C_Small C?
+L Device:C_Small C4
 U 1 1 5FFB2B3F
 P 2800 1550
-F 0 "C?" H 2892 1596 50  0000 L CNN
+F 0 "C4" H 2892 1596 50  0000 L CNN
 F 1 "10uF" H 2892 1505 50  0000 L CNN
-F 2 "" H 2800 1550 50  0001 C CNN
+F 2 "Capacitor_SMD:C_0805_2012Metric_Pad1.18x1.45mm_HandSolder" H 2800 1550 50  0001 C CNN
 F 3 "~" H 2800 1550 50  0001 C CNN
 	1    2800 1550
@@
 $EndComp
 $Comp
-L Regulator_Linear:XC6220B331MR U?
+L Regulator_Linear:XC6220B331MR U1
 U 1 1 5FE8C427
 P 2150 1500
-F 0 "U?" H 2150 1867 50  0000 C CNN
+F 0 "U1" H 2150 1867 50  0000 C CNN
 F 1 "XC6220B331MR" H 2150 1776 50  0000 C CNN
 F 2 "Package_TO_SOT_SMD:SOT-23-5" H 2150 1500 50  0001 C CNN
@@
 	2500 3500 2500 3900
 $Comp
-L Device:C_Small C?
+L Device:C_Small C2
 U 1 1 600095DC
 P 1400 3750
-F 0 "C?" H 1492 3796 50  0000 L CNN
+F 0 "C2" H 1492 3796 50  0000 L CNN
 F 1 "0.1uF" H 1492 3705 50  0000 L CNN
-F 2 "" H 1400 3750 50  0001 C CNN
+F 2 "Capacitor_SMD:C_0603_1608Metric_Pad1.08x0.95mm_HandSolder" H 1400 3750 50  0001 C CNN
 F 3 "~" H 1400 3750 50  0001 C CNN
 	1    1400 3750
@@
 GPIO14
 Text Label 2450 6000 0    50   ~ 0
-GPIO23
+GPIO15
 Text Label 4300 3800 0    50   ~ 0
 GPIO0
@@
 	7300 5250 7650 5250
 Wire Wire Line
-	7300 5150 7650 5150
-Wire Wire Line
 	7300 5050 7650 5050
 Wire Wire Line
@@
 GPIO25
 $Comp
-L Connector:Conn_01x05_Male J?
-U 1 1 5FE8BD4D
-P 7850 4150
-F 0 "J?" H 8250 4600 50  0000 R CNN
-F 1 "Conn_01x05_Male" H 8250 4500 50  0000 R CNN
-F 2 "" H 7850 4150 50  0001 C CNN
-F 3 "~" H 7850 4150 50  0001 C CNN
-	1    7850 4150
-	-1   0    0    -1
-$EndComp
-$Comp
-L Connector:Conn_01x10_Male J?
+L Connector:Conn_01x10_Male J3
 U 1 1 5FE8D4C8
 P 8800 5250
-F 0 "J?" H 9350 5900 50  0000 R CNN
+F 0 "J3" H 9350 5900 50  0000 R CNN
 F 1 "Conn_01x10_Male" H 9350 5800 50  0000 R CNN
-F 2 "" H 8800 5250 50  0001 C CNN
+F 2 "Connector_PinHeader_2.54mm:PinHeader_1x10_P2.54mm_Vertical" H 8800 5250 50  0001 C CNN
 F 3 "~" H 8800 5250 50  0001 C CNN
 	1    8800 5250
@@
 $EndComp
 $Comp
-L Connector:Conn_01x10_Male J?
+L Connector:Conn_01x10_Male J2
 U 1 1 5FE8CA6B
 P 7850 5250
-F 0 "J?" H 8400 5900 50  0000 R CNN
+F 0 "J2" H 8400 5900 50  0000 R CNN
 F 1 "Conn_01x10_Male" H 8400 5800 50  0000 R CNN
-F 2 "" H 7850 5250 50  0001 C CNN
+F 2 "Connector_PinHeader_2.54mm:PinHeader_1x10_P2.54mm_Vertical" H 7850 5250 50  0001 C CNN
 F 3 "~" H 7850 5250 50  0001 C CNN
 	1    7850 5250
@@
 	7100 5650 7650 5650
 $Comp
-L power:GND #PWR?
+L power:GND #PWR0113
 U 1 1 600E79DD
 P 8100 4900
-F 0 "#PWR?" H 8100 4650 50  0001 C CNN
+F 0 "#PWR0113" H 8100 4650 50  0001 C CNN
 F 1 "GND" H 8105 4727 50  0000 C CNN
 F 2 "" H 8100 4900 50  0001 C CNN
@@
 Text Label 8250 5750 0    50   ~ 0
 GPIO23
+Wire Wire Line
+	7650 5150 7300 5150
+Wire Wire Line
+	4250 4900 4550 4900
+Wire Wire Line
+	4550 4600 4250 4600
+Text Label 4300 4900 0    50   ~ 0
+GPIO22
+Text Label 4300 4600 0    50   ~ 0
+GPIO21
+$Comp
+L Connector:Conn_01x04_Male J1
+U 1 1 5FE8BD4D
+P 7850 4150
+F 0 "J1" H 8250 4550 50  0000 R CNN
+F 1 "Conn_01x04_Male" H 8250 4450 50  0000 R CNN
+F 2 "Connector_PinHeader_2.54mm:PinHeader_1x04_P2.54mm_Vertical" H 7850 4150 50  0001 C CNN
+F 3 "~" H 7850 4150 50  0001 C CNN
+	1    7850 4150
+	-1   0    0    -1
+$EndComp
 $EndSCHEMATC

Commit message: First routing done
Parts:
- removed C2: 0.1uF, Capacitor_SMD:C_0603_1608Metric_Pad1.08x0.95mm_HandSolder, symbol Device:C_Small
- added R1: 10k, Resistor_SMD:R_0603_1608Metric_Pad0.98x0.95mm_HandSolder, symbol Device:R_Small
- J1: value Conn_01x04_Male -> Conn_01x06_Male; footprint Connector_PinHeader_2.54mm:PinHeader_1x04_P2.54mm_Vertical -> B6B-ZR(LF)(SN):JST_B6B-ZR(LF)(SN); symbol Connector:Conn_01x04_Male -> Connector:Conn_01x06_Male
Connections:
- net labels added: GPIO2
- net labels removed: GPIO35
- wire segments 103 -> 111
Other:
- moved on the sheet: C3, J2, J3
